Commit message: katana_controller/gazebo(Migrate)-  katana driver to ROS 2, update URDF meshes, and add Gazebo support.

File: katana_description/urdf/gazebo.urdf.xacro (robot description, xacro)
@@ -2,27 +2,7 @@
 <robot xmlns:xacro="http://ros.org/wiki/xacro">
   <gazebo>
-    <plugin name="gazebo_ros_control" filename="libgazebo_ros_control.so">
-      <robotSimType>gazebo_ros_control/DefaultRobotHWSim</robotSimType>
+    <plugin filename="ign_ros2_control-system" name="ign_ros2_control::IgnitionROS2ControlPlugin">
+      <parameters>$(find katana_arm_gazebo)/config/katana_controllers.yaml</parameters>
     </plugin>
-    <!-- gripper controller -->
-    <plugin name="katana_gripper_controller" filename="libgazebo_ros_katana_gripper.so">
-      <alwaysOn>true</alwaysOn>
-      <node_namespace>katana</node_namespace>
-      <r_finger_joint>katana_r_finger_joint</r_finger_joint>
-      <l_finger_joint>katana_l_finger_joint</l_finger_joint>
-      <updateRate>1000.0</updateRate>
-      <max_torque>0.5</max_torque>
-    </plugin>
-    <!-- a formal implementation of grasp hack in gazebo with fixed joint -->
-    <gripper name="katana_gripper_grasp_hack">
-      <grasp_check>
-        <attach_steps>20</attach_steps>
-        <detach_steps>40</detach_steps>
-        <min_contact_count>2</min_contact_count>
-      </grasp_check>
-      <gripper_link>katana_r_finger_link</gripper_link>
-      <gripper_link>katana_l_finger_link</gripper_link>
-      <palm_link>katana_gripper_link</palm_link>
-    </gripper>
   </gazebo>
   <!-- NOTE: all gazebo extensions are listed here: simulator_gazebo/gazebo/src/urdf2gazebo.cpp -->

File: katana_description/urdf/katana_450_6m90a.urdf.xacro (robot description, xacro)
@@ -32,5 +32,5 @@
       <origin xyz="0 0 0" rpy="0 0 0" />
       <geometry>
-        <mesh filename="package://katana_description/meshes/katana/convex/katana_base_link_convex.stl"/>
+        <mesh filename="package://katana_description/meshes/katana/katana_base_link.stl"/>
       </geometry>
     </collision>
@@ -62,5 +62,5 @@
       <origin xyz="0 0 ${-base_height}" rpy="0 0 0" />
       <geometry>
-        <mesh filename="package://katana_description/meshes/katana/convex/katana_motor1_pan_link_convex.stl"/>
+        <mesh filename="package://katana_description/meshes/katana/katana_motor1_pan_link.stl"/>
       </geometry>
     </collision>
@@ -96,5 +96,5 @@
         <origin rpy="${-M_PI/2} 0 0" xyz="0 0 0"/>
         <geometry>
-          <mesh filename="package://katana_description/meshes/katana/convex/katana_motor2_lift_link_convex.stl"/>
+          <mesh filename="package://katana_description/meshes/katana/katana_motor2_lift_link.stl"/>
         </geometry>
       </collision>
@@ -131,5 +131,5 @@
         <origin rpy="${-M_PI/2} 0 0" xyz="0 0 0"/>
         <geometry>
-          <mesh filename="package://katana_description/meshes/katana/convex/katana_motor3_lift_link_convex.stl"/>
+          <mesh filename="package://katana_description/meshes/katana/katana_motor3_lift_link.stl"/>
         </geometry>
       </collision>
@@ -165,5 +165,5 @@
         <origin rpy="${M_PI/2} 0 0" xyz="0 0 0"/>
         <geometry>
-          <mesh filename="package://katana_description/meshes/katana/convex/katana_motor4_lift_link_convex.stl"/>
+          <mesh filename="package://katana_description/meshes/katana/katana_motor4_lift_link.stl"/>
         </geometry>
       </collision>
@@ -199,5 +199,5 @@
         <origin rpy="0 ${M_PI/2} 0" xyz="0 0 0"/>
         <geometry>
-          <mesh filename="package://katana_description/meshes/katana/convex/katana_motor5_wrist_roll_link_convex.stl"/>
+          <mesh filename="package://katana_description/meshes/katana/katana_motor5_wrist_roll_link.stl"/>
         </geometry>
       </collision>
@@ -226,5 +226,5 @@
         <origin rpy="0 ${M_PI} 0" xyz="0 0 0"/>
         <geometry>
-          <mesh filename="package://katana_description/meshes/katana/convex/katana_gripper_link_convex.stl"/>
+          <mesh filename="package://katana_description/meshes/katana/katana_gripper_link.stl"/>
         </geometry>
       </collision>
@@ -255,5 +255,5 @@
           <origin rpy="0 ${M_PI} 0" xyz="0 0 0"/>
           <geometry>
-            <mesh filename="package://katana_description/meshes/katana/convex/katana_gripper_${prefix}_finger_convex.stl"/>
+            <mesh filename="package://katana_description/meshes/katana/katana_gripper_${prefix}_finger.stl"/>
           </geometry>
         </collision>

File: katana_description/urdf/transmissions.urdf.xacro (robot description, xacro)
@@ -1,23 +1,24 @@
 <?xml version="1.0"?>
 <robot xmlns:xacro="http://ros.org/wiki/xacro">
-  <!-- transmissions are required by the controller manager (here: for simulation in gazebo) -->
-  <xacro:macro name="katana_transmission" params="name">
-    <transmission name="${name}_trans">
-      <type>transmission_interface/SimpleTransmission</type>
-      <joint name="${name}_joint">
-        <hardwareInterface>EffortJointInterface</hardwareInterface>
+  <ros2_control name="KatanaHardware" type="system">
+    <hardware>
+      <plugin>gz_ros2_control/GazeboSimSystem</plugin>
+    </hardware>
+    <xacro:macro name="katana_joint_interface" params="name initial_pos">
+      <joint name="${name}">
+        <command_interface name="position"/>
+        <state_interface name="position">
+          <param name="initial_value">${initial_pos}</param>
+        </state_interface>
+        <state_interface name="velocity"/>
       </joint>
-      <actuator name="${name}_motor">
-        <hardwareInterface>EffortJointInterface</hardwareInterface>
-        <mechanicalReduction>1</mechanicalReduction>
-      </actuator>
-    </transmission>
-  </xacro:macro>
-  <xacro:katana_transmission name="katana_motor1_pan" />
-  <xacro:katana_transmission name="katana_motor2_lift" />
-  <xacro:katana_transmission name="katana_motor3_lift" />
-  <xacro:katana_transmission name="katana_motor4_lift" />
-  <xacro:katana_transmission name="katana_motor5_wrist_roll" />
-  <xacro:katana_transmission name="katana_r_finger" />
-  <xacro:katana_transmission name="katana_l_finger" />
+    </xacro:macro>
+    <xacro:katana_joint_interface name="katana_motor1_pan_joint" initial_pos="-3.022" />
+    <xacro:katana_joint_interface name="katana_motor2_lift_joint" initial_pos="2.163" />
+    <xacro:katana_joint_interface name="katana_motor3_lift_joint" initial_pos="-2.207" />
+    <xacro:katana_joint_interface name="katana_motor4_lift_joint" initial_pos="-2.026" />
+    <xacro:katana_joint_interface name="katana_motor5_wrist_roll_joint" initial_pos="-2.990" />
+    <xacro:katana_joint_interface name="katana_r_finger_joint" initial_pos="0.3" />
+    <xacro:katana_joint_interface name="katana_l_finger_joint" initial_pos="0.3" />
+  </ros2_control>
 </robot>

Commit message: moveit2(Migrate): initialize MoveIt 2 configuration package

File: katana_description/urdf/gazebo.urdf.xacro (robot description, xacro)
@@ -1,9 +1,12 @@
 <?xml version="1.0"?>
 <robot xmlns:xacro="http://ros.org/wiki/xacro">
-  <gazebo>
-    <plugin filename="ign_ros2_control-system" name="ign_ros2_control::IgnitionROS2ControlPlugin">
-      <parameters>$(find katana_arm_gazebo)/config/katana_controllers.yaml</parameters>
-    </plugin>
-  </gazebo>
+  <xacro:arg name="use_gazebo" default="false"/>
+  <xacro:if value="${'$(arg use_gazebo)' == 'true'}">
+    <gazebo>
+      <plugin filename="ign_ros2_control-system" name="ign_ros2_control::IgnitionROS2ControlPlugin">
+        <parameters>$(find katana_arm_gazebo)/config/katana_controllers.yaml</parameters>
+      </plugin>
+    </gazebo>
+  </xacro:if>
   <!-- NOTE: all gazebo extensions are listed here: simulator_gazebo/gazebo/src/urdf2gazebo.cpp -->
   <!-- all materials are listed here: simulator_gazebo/gazebo/gazebo/share/gazebo/Media/materials/ -->

File: katana_description/urdf/katana_450_6m90a.urdf.xacro (robot description, xacro)
@@ -2,6 +2,9 @@
 <robot xmlns:xacro="http://ros.org/wiki/xacro"
        name="katana_450_6m90a">
-  <xacro:include filename="$(find katana_description)/urdf/transmissions.urdf.xacro"/>
-  <xacro:include filename="$(find katana_description)/urdf/gazebo.urdf.xacro"/>
+  <xacro:arg name="use_gazebo" default="false"/>
+  <xacro:if value="${'$(arg use_gazebo)' == 'true'}">
+    <xacro:include filename="$(find katana_description)/urdf/transmissions.urdf.xacro"/>
+    <xacro:include filename="$(find katana_description)/urdf/gazebo.urdf.xacro"/>
+  </xacro:if>
   <xacro:property name="M_PI" value="3.1415926535897931" />
   <!-- all values from the katana manual -->

File: katana_description/urdf/transmissions.urdf.xacro (robot description, xacro)
@@ -1,24 +1,27 @@
 <?xml version="1.0"?>
 <robot xmlns:xacro="http://ros.org/wiki/xacro">
-  <ros2_control name="KatanaHardware" type="system">
-    <hardware>
-      <plugin>gz_ros2_control/GazeboSimSystem</plugin>
-    </hardware>
-    <xacro:macro name="katana_joint_interface" params="name initial_pos">
-      <joint name="${name}">
-        <command_interface name="position"/>
-        <state_interface name="position">
-          <param name="initial_value">${initial_pos}</param>
-        </state_interface>
-        <state_interface name="velocity"/>
-      </joint>
-    </xacro:macro>
-    <xacro:katana_joint_interface name="katana_motor1_pan_joint" initial_pos="-3.022" />
-    <xacro:katana_joint_interface name="katana_motor2_lift_joint" initial_pos="2.163" />
-    <xacro:katana_joint_interface name="katana_motor3_lift_joint" initial_pos="-2.207" />
-    <xacro:katana_joint_interface name="katana_motor4_lift_joint" initial_pos="-2.026" />
-    <xacro:katana_joint_interface name="katana_motor5_wrist_roll_joint" initial_pos="-2.990" />
-    <xacro:katana_joint_interface name="katana_r_finger_joint" initial_pos="0.3" />
-    <xacro:katana_joint_interface name="katana_l_finger_joint" initial_pos="0.3" />
-  </ros2_control>
+  <xacro:arg name="use_gazebo" default="false"/>
+  <xacro:if value="${'$(arg use_gazebo)' == 'true'}">
+    <ros2_control name="KatanaHardware" type="system">
+      <hardware>
+        <plugin>gz_ros2_control/GazeboSimSystem</plugin>
+      </hardware>
+      <xacro:macro name="katana_joint_interface" params="name initial_pos">
+        <joint name="${name}">
+          <command_interface name="position"/>
+          <state_interface name="position">
+            <param name="initial_value">${initial_pos}</param>
+          </state_interface>
+          <state_interface name="velocity"/>
+        </joint>
+      </xacro:macro>
+      <xacro:katana_joint_interface name="katana_motor1_pan_joint" initial_pos="-3.022" />
+      <xacro:katana_joint_interface name="katana_motor2_lift_joint" initial_pos="2.163" />
+      <xacro:katana_joint_interface name="katana_motor3_lift_joint" initial_pos="-2.207" />
+      <xacro:katana_joint_interface name="katana_motor4_lift_joint" initial_pos="-2.026" />
+      <xacro:katana_joint_interface name="katana_motor5_wrist_roll_joint" initial_pos="-2.990" />
+      <xacro:katana_joint_interface name="katana_r_finger_joint" initial_pos="0.3" />
+      <xacro:katana_joint_interface name="katana_l_finger_joint" initial_pos="0.3" />
+    </ros2_control>
+  </xacro:if>
 </robot>
