Commit message: katana_moveit2(refactor/feat): add MoveIt configuration package for the 400 version(i used the wrong urdf the whole time) and update hardware interface for ROS 2 control integration

File: katana_description/urdf/controlbox.urdf.xacro (robot description, xacro)
@@ -1,6 +1,6 @@
 <?xml version="1.0"?>
 <robot xmlns:xacro="http://ros.org/wiki/xacro" >
-  <property name="M_PI" value="3.1415926535897931" />
-  <property name="controlbox_height" value="0.073" />
+  <xacro:property name="M_PI" value="3.1415926535897931" />
+  <xacro:property name="controlbox_height" value="0.073" />
   <link name="katana_internal_controlbox_link">
     <visual>
@@ -32,6 +32,3 @@
     <origin xyz="0 0 ${controlbox_height}"/>
   </joint>
-  <gazebo reference="katana_internal_controlbox_link">
-    <material value="Gazebo/Grey" />
-  </gazebo>
 </robot>

File: katana_description/urdf/katana_400_6m180.urdf.xacro (robot description, xacro)
@@ -2,13 +2,16 @@
 <robot xmlns:xacro="http://ros.org/wiki/xacro"
   name="katana_400_6m180">
-  <xacro:include filename="$(find katana_description)/urdf/transmissions.urdf.xacro"/>
-  <xacro:include filename="$(find katana_description)/urdf/gazebo.urdf.xacro"/>
-  <property name="M_PI" value="3.1415926535897931" />
+  <xacro:arg name="use_gazebo" default="false"/>
+  <xacro:if value="${'$(arg use_gazebo)' == 'true'}">
+    <xacro:include filename="$(find katana_description)/urdf/transmissions.urdf.xacro"/>
+    <xacro:include filename="$(find katana_description)/urdf/gazebo.urdf.xacro"/>
+  </xacro:if>
+  <xacro:property name="M_PI" value="3.1415926535897931" />
   <!-- all values from the katana manual -->
-  <property name="base_height" value="0.2015" />
-  <property name="link2_length" value="0.19" />
-  <property name="link3_length" value="0.139" />
-  <property name="link4_length" value="0.1523" />
-  <property name="link5_length" value="0.1505" />
+  <xacro:property name="base_height" value="0.2015" />
+  <xacro:property name="link2_length" value="0.19" />
+  <xacro:property name="link3_length" value="0.191" />
+  <xacro:property name="link4_length" value="0.1523" />
+  <xacro:property name="link5_length" value="0.1505" />
   <!-- All inertial values (mass, center of mass and inertia tensor) have been
        calculated from the meshes using MeshLab -->
@@ -31,5 +34,5 @@
       <origin xyz="0 0 0" rpy="0 0 0" />
       <geometry>
-        <mesh filename="package://katana_description/meshes/katana/convex/katana_base_link_convex.stl"/>
+        <mesh filename="package://katana_description/meshes/katana/katana_base_link.stl"/>
       </geometry>
     </collision>
@@ -61,5 +64,5 @@
       <origin xyz="0 0 ${-base_height}" rpy="0 0 0" />
       <geometry>
-        <mesh filename="package://katana_description/meshes/katana/convex/katana_motor1_pan_link_convex.stl"/>
+        <mesh filename="package://katana_description/meshes/katana/katana_motor1_pan_link.stl"/>
       </geometry>
     </collision>
@@ -95,5 +98,5 @@
         <origin rpy="${-M_PI/2} 0 0" xyz="0 0 0"/>
         <geometry>
-          <mesh filename="package://katana_description/meshes/katana/convex/katana_motor2_lift_link_convex.stl"/>
+          <mesh filename="package://katana_description/meshes/katana/katana_motor2_lift_link.stl"/>
         </geometry>
       </collision>
@@ -130,5 +133,5 @@
         <origin rpy="${-M_PI/2} 0 0" xyz="0 0 0"/>
         <geometry>
-          <mesh filename="package://katana_description/meshes/katana/convex/katana_motor3_lift_link_convex.stl"/>
+          <mesh filename="package://katana_description/meshes/katana/katana_motor3_lift_link.stl"/>
         </geometry>
       </collision>
@@ -164,5 +167,5 @@
         <origin rpy="${M_PI/2} 0 0" xyz="0 0 0"/>
         <geometry>
-          <mesh filename="package://katana_description/meshes/katana/convex/katana_motor4_lift_link_convex.stl"/>
+          <mesh filename="package://katana_description/meshes/katana/katana_motor4_lift_link.stl"/>
         </geometry>
       </collision>
@@ -198,5 +201,5 @@
         <origin rpy="0 ${M_PI} 0" xyz="0 0 0"/>
         <geometry>
-          <mesh filename="package://katana_description/meshes/katana/convex/katana_motor5_wrist_roll_link_convex.stl"/>
+          <mesh filename="package://katana_description/meshes/katana/katana_motor5_wrist_roll_link.stl"/>
         </geometry>
       </collision>
@@ -225,5 +228,5 @@
         <origin rpy="0 ${M_PI} 0" xyz="0 0 0"/>
         <geometry>
-          <mesh filename="package://katana_description/meshes/katana/convex/katana_gripper_link_convex.stl"/>
+          <mesh filename="package://katana_description/meshes/katana/katana_gripper_link.stl"/>
         </geometry>
       </collision>
@@ -254,5 +257,5 @@
           <origin rpy="0 ${M_PI} 0" xyz="0 0 0"/>
           <geometry>
-            <mesh filename="package://katana_description/meshes/katana/convex/katana_gripper_${prefix}_finger_convex.stl"/>
+            <mesh filename="package://katana_description/meshes/katana/katana_gripper_${prefix}_finger.stl"/>
           </geometry>
         </collision>
