Commit message: katana_moveit2(feat): it worked!!!!  ,add full system launch configuration, update joint limits, and refine controller parameters for Katana 400

File: katana_description/urdf/katana_400_6m180.urdf.xacro (robot description, xacro)
@@ -81,5 +81,5 @@
     <origin xyz="0 0 0" rpy="${M_PI/2} 0 0"/>
     <axis xyz="0 0 1"/>
-    <limit effort="0.6" lower="-0.135228" upper="2.168572"  velocity="1.190799"/>
+    <limit effort="0.6" lower="-0.135228" upper="2.20"  velocity="1.190799"/>
   </joint>
   <link name="katana_motor2_lift_link">

Commit message: katana_misc_ik_solver(refactor-feat): move the unrelate module to the related one and create simple low-level IK move from kni lib

File: katana_description/urdf/katana_400_6m180.urdf.xacro (robot description, xacro)
@@ -244,5 +244,5 @@
         <origin rpy="${rotate} 0 0" xyz="0.034 0 0"/>
         <axis xyz="0 0 1"/>
-        <limit effort="0.5" lower="-0.44" upper="0.31"  velocity="0.718834"/>
+        <limit effort="0.5" lower="-0.34" upper="0.31"  velocity="0.718834"/>
       </joint>
       <link name="katana_${prefix}_finger_link">
