Commit message: katana_tests(feat): implement Katana hardware interface improvements, add real hardware support, and introduce diagnostic testing tools.

File: katana_moveit_config/config/katana_450_6m90a.ros2_control.xacro (robot description, xacro)
@@ -1,34 +1,36 @@
 <?xml version="1.0"?>
 <robot xmlns:xacro="http://www.ros.org/wiki/xacro">
-    <xacro:macro name="katana_450_6m90a_ros2_control" params="name initial_positions_file">
+    <!-- connection_type : 'tcp' or 'serial'
+         ip_address     : arm controller IP (TCP mode)
+         tcp_port       : KNI port, default 5566 (TCP mode)
+         serial_port    : port index N for /dev/ttyS<N> (serial mode)
+         serial_baud    : baud rate (serial mode)
+         config_file    : absolute path to the .cfg for your arm variant
+                          e.g. <kni_share>/KNI_4.3.0/configfiles450/katana6M90A_G.cfg
+         calibrate_on_startup : 'true' to run calibration sequence on first activate -->
+    <xacro:macro name="katana_450_6m90a_ros2_control"
+                 params="name initial_positions_file
+                         connection_type
+                         ip_address
+                         tcp_port
+                         serial_port
+                         serial_baud
+                         config_file
+                         calibrate_on_startup">
         <xacro:property name="initial_positions" value="${xacro.load_yaml(initial_positions_file)['initial_positions']}"/>
         <ros2_control name="${name}" type="system">
             <hardware>
-                <!-- <plugin>mock_components/GenericSystem</plugin>-->
-                <!-- Real hardware plugin — connects to the Katana arm over TCP -->
                 <plugin>katana_driver/KatanaHardwareInterface</plugin>
-                <!-- ── Connection parameters ───────────────────────────────────
-                     ip_address   : IP of the Katana controller (set on the arm's
-                                    onboard PC or USB-Ethernet adapter).
-                     config_file  : Absolute path to the .cfg file that matches your
-                                    arm variant (katana6M180_F.cfg or _G.cfg etc.).
-                                    The files live in:
-                                    install/kni/share/kni/KNI_4.3.0/configfiles450/
-                     calibrate_on_startup : set to "false" if the arm is already
-                                           homed and you don't want it to recalibrate.
-                ────────────────────────────────────────────────────────────────                <!-- Connection Parameters -->
-                <param name="connection_type">serial</param> <!-- 'tcp' or 'serial' -->
-                <!-- TCP Params (used if type is 'tcp') -->
-                <param name="ip_address">192.168.1.1</param>
-                <param name="tcp_port">5566</param>
-                <!-- Serial Params (used if type is 'serial') -->
-                <param name="serial_port">0</param> <!-- 0 = /dev/ttyS0, 1 = /dev/ttyS1, etc. -->
-                <param name="serial_baud">57600</param>
-                <param name="config_file">$(find kni)/share/kni/KNI_4.3.0/configfiles450/katana6M180_F.cfg</param>
-                <param name="calibrate_on_startup">true</param>
+                <param name="connection_type">${connection_type}</param>
+                <param name="ip_address">${ip_address}</param>
+                <param name="tcp_port">${tcp_port}</param>
+                <param name="serial_port">${serial_port}</param>
+                <param name="serial_baud">${serial_baud}</param>
+                <param name="config_file">${config_file}</param>
+                <param name="calibrate_on_startup">${calibrate_on_startup}</param>
             </hardware>
             <joint name="katana_motor1_pan_joint">
                 <command_interface name="position"/>
-                <command_interface name="velocity"/>
+                <!-- <command_interface name="velocity"/> -->
                 <state_interface name="position">
                   <param name="initial_value">${initial_positions['katana_motor1_pan_joint']}</param>
@@ -38,5 +40,5 @@
             <joint name="katana_motor2_lift_joint">
                 <command_interface name="position"/>
-                <command_interface name="velocity"/>
+                <!-- <command_interface name="velocity"/> -->
                 <state_interface name="position">
                   <param name="initial_value">${initial_positions['katana_motor2_lift_joint']}</param>
@@ -46,5 +48,5 @@
             <joint name="katana_motor3_lift_joint">
                 <command_interface name="position"/>
-                <command_interface name="velocity"/>
+                <!-- <command_interface name="velocity"/> -->
                 <state_interface name="position">
                   <param name="initial_value">${initial_positions['katana_motor3_lift_joint']}</param>
@@ -54,5 +56,5 @@
             <joint name="katana_motor4_lift_joint">
                 <command_interface name="position"/>
-                <command_interface name="velocity"/>
+                <!-- <command_interface name="velocity"/> -->
                 <state_interface name="position">
                   <param name="initial_value">${initial_positions['katana_motor4_lift_joint']}</param>
@@ -62,5 +64,5 @@
             <joint name="katana_motor5_wrist_roll_joint">
                 <command_interface name="position"/>
-                <command_interface name="velocity"/>
+                <!-- <command_interface name="velocity"/> -->
                 <state_interface name="position">
                   <param name="initial_value">${initial_positions['katana_motor5_wrist_roll_joint']}</param>
@@ -70,5 +72,5 @@
             <joint name="katana_l_finger_joint">
                 <command_interface name="position"/>
-                <command_interface name="velocity"/>
+                <!-- <command_interface name="velocity"/> -->
                 <state_interface name="position">
                   <param name="initial_value">${initial_positions['katana_l_finger_joint']}</param>
@@ -78,5 +80,5 @@
             <joint name="katana_r_finger_joint">
                 <command_interface name="position"/>
-                <command_interface name="velocity"/>
+                <!-- <command_interface name="velocity"/> -->
                 <state_interface name="position">
                   <param name="initial_value">${initial_positions['katana_r_finger_joint']}</param>

File: katana_moveit_config/config/katana_450_6m90a.urdf.xacro (robot description, xacro)
@@ -2,8 +2,25 @@
 <robot xmlns:xacro="http://www.ros.org/wiki/xacro" name="katana_450_6m90a">
     <xacro:arg name="initial_positions_file" default="initial_positions.yaml" />
+    <!-- Hardware connection args — overridden by real_hardware.launch.py -->
+    <xacro:arg name="connection_type"        default="serial" />
+    <xacro:arg name="ip_address"             default="192.168.1.1" />
+    <xacro:arg name="tcp_port"               default="5566" />
+    <xacro:arg name="serial_port"            default="0" />
+    <xacro:arg name="serial_baud"            default="57600" />
+    <xacro:arg name="config_file"            default="$(find kni)/KNI_4.3.0/configfiles450/katana6M90A_G.cfg" />
+    <xacro:arg name="calibrate_on_startup"   default="true" />
     <!-- Import katana_450_6m90a urdf file -->
     <xacro:include filename="$(find katana_description)/urdf/katana_450_6m90a.urdf.xacro" />
     <!-- Import control_xacro -->
     <xacro:include filename="katana_450_6m90a.ros2_control.xacro" />
-    <xacro:katana_450_6m90a_ros2_control name="FakeSystem" initial_positions_file="$(arg initial_positions_file)"/>
+    <xacro:katana_450_6m90a_ros2_control
+        name="KatanaHW"
+        initial_positions_file="$(arg initial_positions_file)"
+        connection_type="$(arg connection_type)"
+        ip_address="$(arg ip_address)"
+        tcp_port="$(arg tcp_port)"
+        serial_port="$(arg serial_port)"
+        serial_baud="$(arg serial_baud)"
+        config_file="$(arg config_file)"
+        calibrate_on_startup="$(arg calibrate_on_startup)" />
 </robot>
