Commit message: rviz_offset(chore): update Katana robot configuration with adjusted joint offsets, limits, and initial positions need to be more precise actually

File: katana400_moveit_config/config/katana_400_6m180_with_controlbox.ros2_control.xacro (robot description, xacro)
@@ -18,9 +18,9 @@
                          config_file
                          calibrate_on_startup
-                         urdf_offset_katana_motor1_pan_joint:=3.0147
-                         urdf_offset_katana_motor2_lift_joint:=0.1508
-                         urdf_offset_katana_motor3_lift_joint:=4.9553
-                         urdf_offset_katana_motor4_lift_joint:=4.8512
-                         urdf_offset_katana_motor5_wrist_roll_joint:=3.8913
+                         urdf_offset_katana_motor1_pan_joint:=0.8290
+                         urdf_offset_katana_motor2_lift_joint:=2.3208
+                         urdf_offset_katana_motor3_lift_joint:=2.7353
+                         urdf_offset_katana_motor4_lift_joint:=2.8212
+                         urdf_offset_katana_motor5_wrist_roll_joint:=0.9013
                          urdf_offset_katana_l_finger_joint:=1.5927
                          urdf_offset_katana_r_finger_joint:=0.0

File: katana_description/urdf/katana_400_6m180.urdf.xacro (robot description, xacro)
@@ -51,5 +51,5 @@
     <origin xyz="0 0 ${base_height}" rpy="0 0 0"/>
     <axis xyz="0 0 1"/>
-    <limit effort="1.5" lower="-3.025528" upper="2.891097" velocity="2.208932"/>
+    <limit effort="1.5" lower="-3.05" upper="2.891097" velocity="2.208932"/>
   </joint>
   <link name="katana_motor1_pan_link">

Commit message: katana_gripper(feat): fix gripper command becuz gripper cant use with splineMovemoent so use moveMotorToEnc instead

File: katana400_moveit_config/config/katana_400_6m180_with_controlbox.ros2_control.xacro (robot description, xacro)
@@ -23,5 +23,5 @@
                          urdf_offset_katana_motor4_lift_joint:=2.9095
                          urdf_offset_katana_motor5_wrist_roll_joint:=0.9013
-                         urdf_offset_katana_l_finger_joint:=1.5927
+                         urdf_offset_katana_l_finger_joint:=0.7040
                          urdf_offset_katana_r_finger_joint:=0.0
                          urdf_flip_katana_motor1_pan_joint:=-1.0
@@ -30,5 +30,5 @@
                          urdf_flip_katana_motor4_lift_joint:=-1.0
                          urdf_flip_katana_motor5_wrist_roll_joint:=-1.0
-                         urdf_flip_katana_l_finger_joint:=1.0
+                         urdf_flip_katana_l_finger_joint:=0.3255
                          urdf_flip_katana_r_finger_joint:=1.0">
         <xacro:property name="initial_positions" value="${xacro.load_yaml(initial_positions_file)['initial_positions']}"/>

File: katana_description/urdf/katana_400_6m180.urdf.xacro (robot description, xacro)
@@ -244,5 +244,5 @@
         <origin rpy="${rotate} 0 0" xyz="0.034 0 0"/>
         <axis xyz="0 0 1"/>
-        <limit effort="0.5" lower="-0.44" upper="0.30"  velocity="0.718834"/>
+        <limit effort="0.5" lower="-0.44" upper="0.31"  velocity="0.718834"/>
       </joint>
       <link name="katana_${prefix}_finger_link">

Commit message: katana_gripper(fix):make gripper use open/close gripper command instead of movetoENc becuz it broke

File: katana400_moveit_config/config/katana_400_6m180_with_controlbox.ros2_control.xacro (robot description, xacro)
@@ -31,5 +31,7 @@
                          urdf_flip_katana_motor5_wrist_roll_joint:=-1.0
                          urdf_flip_katana_l_finger_joint:=0.3255
-                         urdf_flip_katana_r_finger_joint:=1.0">
+                         urdf_flip_katana_r_finger_joint:=1.0
+                         gripper_open_enc:=30770
+                         gripper_close_enc:=18000">
         <xacro:property name="initial_positions" value="${xacro.load_yaml(initial_positions_file)['initial_positions']}"/>
         <ros2_control name="${name}" type="system">
@@ -57,4 +59,6 @@
                 <param name="urdf_flip_katana_l_finger_joint">${urdf_flip_katana_l_finger_joint}</param>
                 <param name="urdf_flip_katana_r_finger_joint">${urdf_flip_katana_r_finger_joint}</param>
+                <param name="gripper_open_enc">${gripper_open_enc}</param>
+                <param name="gripper_close_enc">${gripper_close_enc}</param>
             </hardware>
             <joint name="katana_motor1_pan_joint">

File: katana_description/urdf/katana_400_6m180.urdf.xacro (robot description, xacro)
@@ -244,5 +244,5 @@
         <origin rpy="${rotate} 0 0" xyz="0.034 0 0"/>
         <axis xyz="0 0 1"/>
-        <limit effort="0.5" lower="-0.34" upper="0.31"  velocity="0.718834"/>
+        <limit effort="0.5" lower="-0.46" upper="0.31"  velocity="0.718834"/>
       </joint>
       <link name="katana_${prefix}_finger_link">

Commit message: katana_gripper(fix):make gripper has just 1 joint and mirror the opposite joint instead for rviz and control

File: katana400_moveit_config/config/katana_400_6m180_with_controlbox.ros2_control.xacro (robot description, xacro)
@@ -24,5 +24,4 @@
                          urdf_offset_katana_motor5_wrist_roll_joint:=0.9013
                          urdf_offset_katana_l_finger_joint:=0.7040
-                         urdf_offset_katana_r_finger_joint:=0.0
                          urdf_flip_katana_motor1_pan_joint:=-1.0
                          urdf_flip_katana_motor2_lift_joint:=-1.0
@@ -31,5 +30,4 @@
                          urdf_flip_katana_motor5_wrist_roll_joint:=-1.0
                          urdf_flip_katana_l_finger_joint:=0.3255
-                         urdf_flip_katana_r_finger_joint:=1.0
                          gripper_open_enc:=30770
                          gripper_close_enc:=18500">
@@ -51,5 +49,4 @@
                 <param name="urdf_offset_katana_motor5_wrist_roll_joint">${urdf_offset_katana_motor5_wrist_roll_joint}</param>
                 <param name="urdf_offset_katana_l_finger_joint">${urdf_offset_katana_l_finger_joint}</param>
-                <param name="urdf_offset_katana_r_finger_joint">${urdf_offset_katana_r_finger_joint}</param>
                 <param name="urdf_flip_katana_motor1_pan_joint">${urdf_flip_katana_motor1_pan_joint}</param>
                 <param name="urdf_flip_katana_motor2_lift_joint">${urdf_flip_katana_motor2_lift_joint}</param>
@@ -58,5 +55,4 @@
                 <param name="urdf_flip_katana_motor5_wrist_roll_joint">${urdf_flip_katana_motor5_wrist_roll_joint}</param>
                 <param name="urdf_flip_katana_l_finger_joint">${urdf_flip_katana_l_finger_joint}</param>
-                <param name="urdf_flip_katana_r_finger_joint">${urdf_flip_katana_r_finger_joint}</param>
                 <param name="gripper_open_enc">${gripper_open_enc}</param>
                 <param name="gripper_close_enc">${gripper_close_enc}</param>
@@ -104,11 +100,4 @@
                 <state_interface name="velocity"/>
             </joint>
-            <joint name="katana_r_finger_joint">
-                <command_interface name="position"/>
-                <state_interface name="position">
-                  <param name="initial_value">${initial_positions['katana_r_finger_joint']}</param>
-                </state_interface>
-                <state_interface name="velocity"/>
-            </joint>
         </ros2_control>
     </xacro:macro>

File: katana_description/urdf/katana_400_6m180.urdf.xacro (robot description, xacro)
@@ -238,5 +238,5 @@
           izz="0.000011290" /></inertial>
     </link>
-    <xacro:macro name="finger" params="prefix rotate">
+    <xacro:macro name="finger" params="prefix rotate mimic:=''">
       <joint name="katana_${prefix}_finger_joint" type="revolute">
         <parent link="katana_gripper_link" />
@@ -245,4 +245,7 @@
         <axis xyz="0 0 1"/>
         <limit effort="0.5" lower="-0.46" upper="0.31"  velocity="0.718834"/>
+        <xacro:unless value="${mimic == ''}">
+          <mimic joint="${mimic}" multiplier="1.0" offset="0.0"/>
+        </xacro:unless>
       </joint>
       <link name="katana_${prefix}_finger_link">
@@ -269,5 +272,5 @@
       </link>
     </xacro:macro>
-    <xacro:finger prefix="r" rotate="0" />
+    <xacro:finger prefix="r" rotate="0" mimic="katana_l_finger_joint" />
     <xacro:finger prefix="l" rotate="${M_PI}" />
     <joint name="katana_gripper_tool_frame_joint" type="fixed">
