Commit message: checkpoint-can run sim

File: description/katana_description/urdf/controlbox.urdf.xacro (robot description, xacro)
@@ -16,5 +16,5 @@
       <origin xyz="0 0 0" rpy="0 0 ${M_PI}" />
       <geometry>
-        <mesh filename="package://katana_description/meshes/katana/convex/katana_internal_controlbox_convex.stl" />
+        <mesh filename="package://katana_description/meshes/katana/katana_internal_controlbox.stl" />
       </geometry>
     </collision>

File: description/mobile_katana_description/urdf/controlbox.urdf.xacro (robot description, xacro)
@@ -14,5 +14,5 @@
       <origin xyz="0 0 0" rpy="0 0 ${M_PI}" />
       <geometry>
-        <mesh filename="package://katana_description/meshes/katana/convex/katana_internal_controlbox_convex.stl" />
+        <mesh filename="package://katana_description/meshes/katana/katana_internal_controlbox.stl" />
       </geometry>
     </collision>
